File: PCB/Retro/Retro.kicad_sch (KiCad schematic)
At the start: 27 parts, among them J1 KeyBoard 5,Rd,Ld,D7..0,Gnd, J2 PortB, J3 PortA, J4 COM: Gnd,Rx,Tx,Rts,Dcd,Cts,5v, J5 Conn_01x20_Pin, J6 Conn_01x20_Pin, J7 Conn_01x20_Pin, SW1 SW_Push, U1 74LS92, U10 GAL20V8B-10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

Commit message: PCB-20250923-0955
Parts:
- removed J5, J6, J7: Conn_01x20_Pin, Connector_PinHeader_2.54mm:PinHeader_1x20_P2.54mm_Vertical, symbol Connector:Conn_01x20_Pin
Connections:
- net BankWr is gone; now on net +5V: U10.1 (Clk/In14), U10.22 (I/O/Q1)
- net D0: now also U8.9 (D7); no longer U8.2 (D0)
- net D1: now also U8.8 (D6); no longer U8.3 (D1)
- net D2: now also U8.7 (D5); no longer U8.4 (D2)
- net D3: now also U8.6 (D4); no longer U8.5 (D3)
- net D4: now also U8.5 (D3); no longer U8.6 (D4)
- net D5: now also U8.4 (D2); no longer U8.7 (D5)
- net D6: now also U8.3 (D1); no longer U8.8 (D6)
- net D7: now also U8.2 (D0); no longer U8.9 (D7)
- net KB0: no longer names the net of J1.2 (Pin_2)
- net KB0: now also U8.12 (Q7); no longer U8.19 (Q0)
- net KB1: no longer names the net of J1.3 (Pin_3)
- net KB1: now also U8.13 (Q6); no longer U8.18 (Q1)
- net KB2: no longer names the net of J1.4 (Pin_4)
- net KB2: now also U8.14 (Q5); no longer U8.17 (Q2)
- net KB3: no longer names the net of J1.5 (Pin_5)
- net KB3: now also U8.15 (Q4); no longer U8.16 (Q3)
- net KB4: no longer names the net of J1.6 (Pin_6)
- net KB4: now also U8.16 (Q3); no longer U8.15 (Q4)
- net KB5: no longer names the net of J1.7 (Pin_7)
- net KB5: now also U8.17 (Q2); no longer U8.14 (Q5)
- net KB6: no longer names the net of J1.8 (Pin_8)
- net KB6: now also U8.18 (Q1); no longer U8.13 (Q6)
- net KB7: no longer names the net of J1.9 (Pin_9)
- net KB7: now also U8.19 (Q0); no longer U8.12 (Q7)
- net KBRD renamed ~{KEY}
Other:
- moved on the sheet: J1
