File: PCB/Retro/Retro.kicad_sch (KiCad schematic)
At the start: 39 parts, among them J1 KeyBoard 5,Rd,Ld,D7..0,Gnd, J2 PortB, J3 PortA, J4 COM: Gnd,Rx,Tx,Rts,Dcd,Cts,5v, J5 Conn_01x12, J6 Screw_Terminal_01x02, SW1 SW_Push, U1 74LS92, U10 GAL20V8B-10, U11 GAL20V8B-10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

Commit message: RestorePoint
Parts:
- added J7: Conn_01x06_Pin, Connector_PinHeader_2.54mm:PinHeader_1x06_P2.54mm_Vertical, symbol Connector:Conn_01x06_Pin
Connections:
- net +5V: no longer U10.1 (Clk/In14), U10.22 (I/O/Q1)
- net Clk2: now also J7.1 (Pin_1)
- net GND: now also J7.2 (Pin_2)
- net RDY: now also J7.3 (Pin_3)
- net SYNC: now also J7.6 (Pin_6)
- net ~{IRQ}: now also J7.4 (Pin_4)
- net ~{NMI}: now also J7.5 (Pin_5)
- new net BankWr: U10.1 (Clk/In14), U10.22 (I/O/Q1)
Other:
- moved on the sheet: J5
