File: PCB/Retro/Retro.kicad_pcb (KiCad board)
At the start: 2 copper layers, 165.1 x 161.3 mm, 27 parts, among them J1 KeyBoard 5,Rd,Ld,D7..0,Gnd, J2 PortB, J3 PortA, J4 COM: Gnd,Rx,Tx,Rts,Dcd,Cts,5v, J5 Conn_01x20_Pin, J6 Conn_01x20_Pin, J7 Conn_01x20_Pin, SW1 SW_Push, U1 74LS92, U10 GAL20V8B-10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

Commit message: PCB-20250923-0955
Parts:
- removed J5, J6, J7: Conn_01x20_Pin, Connector_PinHeader_2.54mm:PinHeader_1x20_P2.54mm_Vertical
- moved J1 176.9 mm to (172.7, 26.7)
- moved U8 139.0 mm to (149.9, 43.2), turned to 90 degrees
- moved U6 38.6 mm to (147.3, 72.4), turned to 0 degrees
Connections:
- net /BankWr renamed Net-(U10-Clk/In14)
- net /KBRD renamed /~{KEY}
- J1 pad 2: /KB0 -> Net-(J1-Pin_2)
- J1 pad 3: /KB1 -> Net-(J1-Pin_3)
- J1 pad 4: /KB2 -> Net-(J1-Pin_4)
- J1 pad 5: /KB3 -> Net-(J1-Pin_5)
- J1 pad 6: /KB4 -> Net-(J1-Pin_6)
- J1 pad 7: /KB5 -> Net-(J1-Pin_7)
- J1 pad 8: /KB6 -> Net-(J1-Pin_8)
- J1 pad 9: /KB7 -> Net-(J1-Pin_9)
- U8 pad 12: /KB7 -> Net-(J1-Pin_2)
- U8 pad 13: /KB6 -> Net-(J1-Pin_3)
- U8 pad 14: /KB5 -> Net-(J1-Pin_4)
- U8 pad 15: /KB4 -> Net-(J1-Pin_5)
- U8 pad 16: /KB3 -> Net-(J1-Pin_6)
- U8 pad 17: /KB2 -> Net-(J1-Pin_7)
- U8 pad 18: /KB1 -> Net-(J1-Pin_8)
- U8 pad 19: /KB0 -> Net-(J1-Pin_9)
- U8 pad 2: /D0 -> /D7
- U8 pad 3: /D1 -> /D6
- U8 pad 4: /D2 -> /D5
- U8 pad 5: /D3 -> /D4
- U8 pad 6: /D4 -> /D3
- U8 pad 7: /D5 -> /D2
- U8 pad 8: /D6 -> /D1
- U8 pad 9: /D7 -> /D0
Routing:
- net +5V: track 520.7 -> 328.1 mm
- net GND: track 423.1 -> 248.7 mm
- net /A0: track 163.6 -> 55.7 mm, vias 5 -> 2
- net /D4: track 449.7 -> 369.4 mm
- net /D5: track 443.2 -> 369.8 mm, vias 4 -> 2
- net /~{IRQ}: track 87.6 -> 18.6 mm, vias 2 -> 0
- net /D6: track 436.7 -> 370.9 mm, vias 4 -> 2
- net /D7: track 430.6 -> 371.6 mm, vias 4 -> 2
- net /A1: track 74.7 -> 39.2 mm
- net /~{WR}: track 35.6 -> 0.00 mm
- net /~{RD}: track 67.1 -> 31.5 mm
- net /R~{W}: track 35.6 -> 0.00 mm
- net /Clk2: track 35.6 -> 0.00 mm
- net /A3: track 74.7 -> 39.2 mm
- net /A2: track 74.7 -> 39.2 mm
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
Commit message: PC-20250923-1122
Parts:
- moved U11 135.0 mm to (-17.8, 58.4)
- moved RP1 125.0 mm to (-20.3, 152.4)
- moved U3 57.0 mm to (90.8, 160.0), turned to -90 degrees
- moved U10 41.9 mm to (-17.8, 20.3)
- moved U9 34.4 mm to (-5.08, 104.1)
- moved SW1 24.1 mm to (2.54, 91.4)
- moved U1 20.9 mm to (55.9, 160.0)
- moved JP153 20.3 mm to (40.6, 177.8)
- moved JP1843 20.3 mm to (55.9, 177.8)
- moved JP460 20.3 mm to (45.7, 177.8)
- moved JP921 20.3 mm to (50.8, 177.8)
- moved U2 19.8 mm to (99.1, 68.6), turned to 0 degrees
- moved J4 18.0 mm to (137.2, 34.9)
- moved OSC1 10.5 mm to (25.4, 144.8), turned to 0 degrees
Routing:
- net +5V: track 328.1 -> 456.0 mm, vias 2 -> 8
- net GND: track 248.7 -> 357.0 mm, vias 4 -> 6
- net /BaudClk: track 2.54 -> 80.2 mm, vias 0 -> 2
- net /D2: track 330.0 -> 398.7 mm, vias 5 -> 4
- net /D1: track 332.9 -> 398.3 mm, vias 5 -> 4
- net /D0: track 335.1 -> 397.3 mm
- net Net-(JP1843-A): track 0.00 -> 57.9 mm, vias 0 -> 2
- net Net-(J4-Pin_4): track 8.27 -> 58.7 mm, vias 0 -> 2
- net Net-(J4-Pin_5): track 19.7 -> 67.1 mm, vias 2 -> 0
- net Net-(J4-Pin_2): track 0.04 -> 46.8 mm, vias 0 -> 2
- net Net-(J4-Pin_3): track 15.9 -> 59.5 mm, vias 2 -> 4
- net Net-(J4-Pin_6): track 19.7 -> 62.2 mm, vias 2 -> 0
- net /A14: track 40.9 -> 10.5 mm, vias 2 -> 0
- net /D6: track 370.9 -> 401.0 mm
- net /D5: track 369.8 -> 397.7 mm
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
Commit message: Added RST switch and address connector
Parts:
- added J5: Conn_01x12, Connector_PinSocket_2.54mm:PinSocket_1x12_P2.54mm_Vertical, F.Cu at (91.4, 171.4)
- SW1: footprint Button_Switch_THT:KSA_Tactile_SPST -> Library:MiniSwitch
- moved SW1 181.2 mm to (162.6, 176.5), turned to 90 degrees
- moved RP1 123.3 mm to (83.8, 86.4)
- moved U10 120.6 mm to (92.7, 68.6), turned to 180 degrees
- moved U9 120.6 mm to (105.4, 152.4), turned to -90 degrees
- moved U11 90.1 mm to (40.6, 127.0), turned to 180 degrees
- moved U3 52.0 mm to (47.0, 132.1), turned to 0 degrees
- moved RV1 10.1 mm to (96.5, 175.3)
- moved JP153 5.08 mm to (35.6, 177.8), turned to -90 degrees
- moved U1 4.02 mm to (54.6, 163.8)
- moved JP1843 3.81 mm to (59.7, 177.8), turned to -90 degrees
- moved JP460 2.54 mm to (43.2, 177.8), turned to -90 degrees
- moved LCD1 0.23 mm to (100.5, 122.1)
- turned JP921 to -90 degrees
Connections:
- net /~{PORT1} renamed /~{PORT}
- LCD1 pad 1: unconnected-(LCD1-FG-Pad1) -> GND
- LCD1 pad 19: unconnected-(LCD1-FS1-Pad19) -> +5V
- RP1 pad 3: /~{IRQ} -> /~{SO}
- RP1 pad 4: /RDY -> /~{IRQ}
- RP1 pad 5: /~{SO} -> /RDY
- U11 pad 15: /~{PORT3} -> /~{RD}
- U11 pad 16: /~{PORT2} -> /~{WR}
- U11 pad 22: /~{IN} -> /~{KEY}
- U3 pad 2: unconnected-(U3-LE-Pad2) -> GND
- U4 pad 31: unconnected-(U4-~{WE}-Pad31) -> +5V
- U7 pad 24: unconnected-(U7-CS1-Pad24) -> +5V
Routing:
- net GND: track 357.0 -> 733.3 mm, vias 6 -> 23
- net +5V: track 456.0 -> 772.5 mm, vias 8 -> 18
- net /~{RD}: track 31.5 -> 325.8 mm, vias 0 -> 2
- net /Clk2: track 0.00 -> 284.2 mm, vias 0 -> 6
- net /~{WR}: track 0.00 -> 282.8 mm
- net /R~{W}: track 0.00 -> 265.4 mm, vias 0 -> 8
- net /A12: track 38.2 -> 300.0 mm, vias 0 -> 6
- net /A13: track 18.3 -> 266.1 mm, vias 0 -> 8
- net /~{KEY}: track 18.3 -> 261.5 mm, vias 2 -> 6
- net /A3: track 39.2 -> 231.6 mm, vias 0 -> 4
- net /DISP: track 0.00 -> 191.0 mm
- net /~{COM}: track 0.00 -> 189.9 mm, vias 0 -> 4
- net /~{IRQ}: track 0.00 -> 189.2 mm, vias 0 -> 8
- net /A2: track 39.2 -> 227.6 mm, vias 0 -> 4
- net /A1: track 39.2 -> 225.6 mm, vias 0 -> 4
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Other:
- board size 165.1 x 161.3 mm -> 141.4 x 101.8 mm

Commit message: Save point
Parts:
- added C1: C, Capacitor_THT:C_Disc_D7.5mm_W2.5mm_P5.00mm, F.Cu at (61.0, 173.3)
- added C10: C, Capacitor_THT:C_Disc_D7.5mm_W2.5mm_P5.00mm, F.Cu at (85.0, 80.6)
- added C11: C, Capacitor_THT:C_Rect_L11.0mm_W2.8mm_P10.00mm_MKT, F.Cu at (29.3, 97.2)
- added C12: C_Polarized_Small, Capacitor_THT:CP_Radial_D10.0mm_P7.50mm, F.Cu at (26.7, 71.6)
- added C13: C_Polarized_Small, Capacitor_THT:CP_Radial_D10.0mm_P7.50mm, F.Cu at (99.1, 174.4)
- added C2: C, Capacitor_THT:C_Rect_L11.0mm_W2.8mm_P10.00mm_MKT, F.Cu at (94.0, 93.3)
- added C3: C, Capacitor_THT:C_Disc_D7.5mm_W2.5mm_P5.00mm, F.Cu at (43.2, 147.7)
- added C4: C, Capacitor_THT:C_Disc_D7.5mm_W2.5mm_P5.00mm, F.Cu at (38.1, 64.1)
- added C5: C, Capacitor_THT:C_Rect_L11.0mm_W2.8mm_P10.00mm_MKT, F.Cu at (38.1, 69.3)
- added C6: C, Capacitor_THT:C_Disc_D7.5mm_W2.5mm_P5.00mm, F.Cu at (152.4, 74.3)
- added C7: C, Capacitor_THT:C_Disc_D7.5mm_W2.5mm_P5.00mm, F.Cu at (177.8, 141.6)
- added C8: C, Capacitor_THT:C_Disc_D7.5mm_W2.5mm_P5.00mm, F.Cu at (176.5, 47.6)
- added C9: C, Capacitor_THT:C_Disc_D7.5mm_W2.5mm_P5.00mm, F.Cu at (99.1, 161.9)
- added J6: Screw_Terminal_01x02, TerminalBlock:TerminalBlock_MaiXu_MX126-5.0-02P_1x02_P5.00mm, F.Cu at (29.3, 32.4)
- J2: moved to F.Cu
- moved RV1 11.2 mm to (104.1, 183.6)
- moved OSC1 9.09 mm to (29.2, 153.0)
- moved J5 8.26 mm to (91.4, 179.7)
- moved U7 8.26 mm to (162.6, 165.7)
- moved LCD1 8.26 mm to (100.5, 130.4)
- moved U8 8.26 mm to (149.9, 51.4)
- moved J1 8.25 mm to (172.7, 34.9)
- moved J2 8.25 mm to (175.3, 137.8), turned to 180 degrees
- moved J3 8.25 mm to (175.3, 173.4)
- moved J4 8.25 mm to (137.2, 43.1)
- moved RP1 8.25 mm to (83.8, 94.6)
- moved SW1 8.25 mm to (162.6, 184.8)
- moved U1 8.25 mm to (54.6, 172.1)
- moved U10 8.25 mm to (92.7, 76.8)
- moved U11 8.25 mm to (40.6, 135.3)
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Connections:
- J5 pad 12: /A12 -> /~{PORT}
- LCD1 pad 22: Net-(LCD1-BLK-Pad22) -> GND
- LCD1 pad 25: Net-(LCD1-BLK-Pad22) -> GND
- RV1 pad 1: Net-(LCD1-BLK-Pad22) -> GND
- U10 pad 6: unconnected-(U10-In05-Pad6) -> /Clk0
Routing:
- net GND: track 733.3 -> 893.3 mm, vias 23 -> 26
- net /Clk0: track 161.7 -> 258.9 mm, vias 2 -> 4
- net /~{PORT}: track 0.00 -> 96.9 mm, vias 0 -> 4
- net /A12: track 300.0 -> 231.1 mm, vias 6 -> 4
- net +5V: track 772.5 -> 822.2 mm
- net /TMR: track 74.0 -> 29.2 mm, vias 3 -> 2
- net /A13: track 266.1 -> 249.9 mm
- net Net-(LCD1-BLK-Pad22): track 14.5 -> 0.00 mm
- net /~{KEY}: track 261.5 -> 269.6 mm
- net Net-(LCD1-VOUT): track 11.8 -> 4.20 mm
- net Net-(LCD1-V0): track 59.2 -> 51.6 mm
- net /~{COM}: track 189.9 -> 196.1 mm
- net /BaudClk: track 236.7 -> 241.8 mm
- net /~{IO}: track 96.9 -> 101.9 mm
- net /A8: track 207.6 -> 204.9 mm
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Other:
- board size 141.4 x 101.8 mm -> 160 x 163 mm
- board text added: "5v GND"
- board text added: "74LS92"
- board text added: "Anton's retro 6502 2025"
- board text added: "CD4059A"
- board text added: "COM 5,Cts,Dcd,Rts,Tx,Rx,Gnd"
- board text added: "COM MC68B50"
- board text added: "CPU 153,460,921,1843 kHz"
- board text added: "EEROM 64k / 128k"
- board text added: "FIX POWER CONNECTOR - SPACE FOR ZIF"
- board text added: "GAL:IO"
- board text added: "GAL:MEM"
- board text added: "KEY 5,Rd,Ld,D7-0,Gnd"
- board text added: "LCD (A0,D7..D0,~{RD}.~{WR} ..)"
- board text added: "PORTA(Gnd,PA0-7,C1,C2,5v)"
- board text added: "PORTB(Gnd,PB0-7,C1,C2,5v)"
- board text added: "R65C02"
- board text added: "RAM 62256"
- board text added: "RESET"
- board text added: "VIA MOS6522"
- board text added: "~{PORT}, A11..A1"

Commit message: RestorePoint
Parts:
- added J7: Conn_01x06_Pin, Connector_PinHeader_2.54mm:PinHeader_1x06_P2.54mm_Vertical, F.Cu at (90.8, 74.4)
- moved J5 5.72 mm to (91.4, 174.0)
- moved LCD1 5.72 mm to (100.5, 124.7)
- moved C4 5.67 mm to (38.7, 58.5)
- moved C1 5.67 mm to (61.6, 167.7)
- moved C10 5.67 mm to (85.7, 75.0)
- moved C11 5.67 mm to (29.9, 91.5)
- moved C13 5.67 mm to (99.7, 168.8)
- moved C2 5.67 mm to (94.6, 87.6)
- moved C3 5.67 mm to (43.8, 142.0)
- moved C5 5.67 mm to (38.7, 63.7)
- moved C6 5.67 mm to (153.0, 68.7)
- moved C7 5.67 mm to (178.4, 136.0)
- moved C8 5.67 mm to (177.1, 41.9)
- moved C9 5.67 mm to (99.7, 156.3)
- moved J2 5.67 mm to (175.9, 132.2)
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Routing:
- net /SYNC: track 0.00 -> 9.19 mm
- net /Clk2: track 286.4 -> 287.0 mm
- net /~{IRQ}: track 189.9 -> 190.4 mm
- net /RDY: track 19.6 -> 19.1 mm
- net GND: track 893.3 -> 892.8 mm
- net /D6: track 390.1 -> 390.6 mm
- net /A8: track 204.9 -> 205.4 mm
- net /A3: track 232.3 -> 232.8 mm
- net /A2: track 227.5 -> 228.1 mm
- net /A10: track 203.6 -> 204.1 mm
- net /A9: track 208.4 -> 209.0 mm
- net /A7: track 188.9 -> 189.4 mm
- net /A4: track 167.5 -> 168.0 mm
- net /A1: track 226.6 -> 227.2 mm
- net /A0: track 234.8 -> 235.3 mm
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Other:
- board size 160 x 163 mm -> 197 x 253 mm
