File: PCB/Mk3/Mk3.kicad_sch (KiCad schematic)
At the start: 44 parts, among them J1 Power, J10 PortA: 5V PA0 PA1 PA2 PA3 PA4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, J2 Bank, J3 Sync ~{NMI} ~{IRQ} RDY Gnd Ph2, J4 PortB: 5V PB0 PB1 PB2 PB3 PB4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, J5 PORT, J6 PORT, J7 PORT, J8 DISPLAY, J9 COM: Gnd,CTS, Vcc, Tx, Rx, DTR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

Commit message: save
Parts:
- added R26: R_Small_US, Resistor_THT:R_Axial_DIN0204_L3.6mm_D1.6mm_P7.62mm_Horizontal, symbol Device:R_Small_US
Connections:
- net +5V: now also R26.1
- net ~{RST}: now also R26.2
Changed lines of the file:
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@@
 	)
 	(junction
+		(at 64.77 44.45)
+		(diameter 0)
+		(color 0 0 0 0)
+	)
+	(junction
 		(at 262.89 22.86)
 		(diameter 0)
@@
 	)
 	(junction
+		(at 64.77 57.15)
+		(diameter 0)
+		(color 0 0 0 0)
+	)
+	(junction
 		(at 81.28 97.79)
 		(diameter 0)
@@
 	(wire
 		(pts
-			(xy 55.88 44.45) (xy 69.85 44.45)
+			(xy 55.88 44.45) (xy 64.77 44.45)
 		)
 		(stroke
@@
 	(wire
 		(pts
+			(xy 64.77 44.45) (xy 69.85 44.45)
+		)
+		(stroke
+			(width 0)
+			(type default)
+		)
+	)
+	(wire
+		(pts
 			(xy 22.86 170.18) (xy 29.21 170.18)
 		)
@@
 	(wire
 		(pts
+			(xy 64.77 53.34) (xy 64.77 57.15)
+		)
+		(stroke
+			(width 0)
+			(type default)
+		)
+	)
+	(wire
+		(pts
 			(xy 271.78 21.59) (xy 271.78 22.86)
 		)
@@
 	(wire
 		(pts
-			(xy 63.5 57.15) (xy 66.04 57.15)
+			(xy 63.5 57.15) (xy 64.77 57.15)
 		)
 		(stroke
@@
 	(wire
 		(pts
+			(xy 64.77 57.15) (xy 66.04 57.15)
+		)
+		(stroke
+			(width 0)
+			(type default)
+		)
+	)
+	(wire
+		(pts
 			(xy 132.08 81.28) (xy 127 81.28)
 		)
@@
 	(wire
 		(pts
+			(xy 64.77 44.45) (xy 64.77 48.26)
+		)
+		(stroke
+			(width 0)
+			(type default)
+		)
+	)
+	(wire
+		(pts
 			(xy 171.45 22.86) (xy 147.32 22.86)
 		)
@@
 	)
 	(symbol
+		(lib_id "Device:R_Small_US")
+		(at 64.77 50.8 0)
+		(unit 1)
+		(exclude_from_sim no)
+		(in_bom yes)
+		(on_board yes)
+		(dnp no)
+		(property "Reference" "R26"
+			(at 66.548 49.022 90)
+			(effects
+				(font
+					(size 1.27 1.27)
+				)
+				(justify left)
+			)
+		)
+		(property "Value" "R_Small_US"
+			(at 67.31 52.0699 0)
+			(effects
+				(font
+					(size 1.27 1.27)
+				)
+				(justify left)
+				(hide yes)
+			)
+		)
+		(property "Footprint" "Resistor_THT:R_Axial_DIN0204_L3.6mm_D1.6mm_P7.62mm_Horizontal"
+			(at 64.77 50.8 0)
+			(effects
+				(font
+					(size 1.27 1.27)
+				)
+				(hide yes)
+			)
+		)
+		(property "Datasheet" "~"
+			(at 64.77 50.8 0)
+			(effects
+				(font
+					(size 1.27 1.27)
+				)
+				(hide yes)
+			)
+		)
+		(property "Description" "Resistor, small US symbol"
+			(at 64.77 50.8 0)
+			(effects
+				(font
+					(size 1.27 1.27)
+				)
+				(hide yes)
+			)
+		)
+		(pin "1"
+		)
+		(pin "2"
+		)
+		(instances
+			(project ""
+				(path "/d41350ce-2040-418d-ae11-f076a5474776"
+					(reference "R26")
+					(unit 1)
+				)
+			)
+		)
+	)
+	(symbol
 		(lib_id "Connector_Generic:Conn_01x32")
 		(at 189.23 149.86 0)
@@
 		(dnp no)
 		(property "Reference" "U2"
-			(at 63.754 48.514 0)
+			(at 59.944 48.26 0)
 			(effects
 				(font
