File: PCB/Mk3/Mk3.kicad_sch (KiCad schematic)
At the start: 45 parts, among them J1 Power, J10 PortA: 5V PA0 PA1 PA2 PA3 PA4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, J2 Bank, J3 Sync ~{NMI} ~{IRQ} RDY Gnd Ph2, J4 PortB: 5V PB0 PB1 PB2 PB3 PB4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, J5 PORT, J6 PORT, J7 PORT, J8 DISPLAY, J9 COM: Gnd,CTS, Vcc, Tx, Rx, DTR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

Commit message: Save point
Parts:
- removed C27: C, Capacitor_THT:C_Disc_D7.5mm_W2.5mm_P5.00mm, symbol Device:C
- removed J7: PORT, Connector_PinSocket_2.54mm:PinSocket_1x32_P2.54mm_Vertical, symbol Connector_Generic:Conn_01x32
- J5: value PORT -> DISPLAY
- J8: value DISPLAY -> PORT
Connections:
- net DISP: now also J5.1 (Pin_1); no longer J8.1 (Pin_1)
- net ~{PORT}: now also J8.1 (Pin_1); no longer J5.1 (Pin_1)
Other:
- moved on the sheet: J6
