File: PCB/Mk4/Mk4.kicad_sch (KiCad schematic)
At the start: 37 parts, among them J1 Power, J2 Bank, J25 HiAddr, J26 Expansion, J27 Conn_01x08_Pin, J3 Sync ~{NMI} ~{IRQ} RDY Gnd Ph2, J5 DISPLAY, SW1 RESET, U1 L7805, U2 DS1813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

Commit message: Latest variation
Other:
- note added: "Mk4"
Changed lines of the file:
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@@
 	(generator_version "9.0")
 	(paper "A4")
+	(text "Mk4"
+		(exclude_from_sim no)
+		(at 17.018 15.494 0)
+		(effects
+			(font
+				(size 2.54 2.54)
+			)
+		)
+	)
 	(junction
 		(at 203.2 49.53)
