File: PCB/Mk5/Mk5.kicad_sch (KiCad schematic)
At the start: 40 parts, among them J1 KeyBoard 5,Rd,Ld,D7..0,Gnd, J2 PortB, J3 PortA, J4 COM: Gnd,Rx,Tx,Rts,Dcd,Cts,5v, J5 Conn_01x12, J6 Screw_Terminal_01x02, J7 Conn_01x06_Pin, SW1 RST, U1 74LS92, U10 GAL20V8B-10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

Commit message: Latest variation
Parts:
- added J8: Conn_01x37_Pin, Connector_PinHeader_2.54mm:PinHeader_1x37_P2.54mm_Vertical, symbol Connector:Conn_01x37_Pin
- added J9: Conn_01x06_Pin, Connector_PinHeader_2.54mm:PinHeader_1x06_P2.54mm_Vertical, symbol Connector:Conn_01x06_Pin
- RV1: footprint Potentiometer_THT:Potentiometer_Runtron_RM-065_Vertical -> Potentiometer_THT:Potentiometer_Piher_PT-15-V15_Vertical
- SW1: footprint Library:MiniSwitch -> Button_Switch_THT:SW_PUSH_1P1T_6x3.5mm_H4.3_APEM_MJTP1243
- U3: footprint Package_DIP:DIP-24_W7.62mm_LongPads -> Package_DIP:DIP-26_W15.24mm_LongPads
Connections:
- net +5V: now also J8.2 (Pin_2)
- net A0: now also J8.24 (Pin_24)
- net A1: now also J8.25 (Pin_25)
- net A10: now also J8.34 (Pin_34)
- net A11: now also J8.35 (Pin_35)
- net A2: now also J8.26 (Pin_26)
- net A3: now also J8.27 (Pin_27)
- net A4: now also J8.28 (Pin_28)
- net A5: now also J8.29 (Pin_29)
- net A6: now also J8.30 (Pin_30)
- net A7: now also J8.31 (Pin_31)
- net A8: now also J8.32 (Pin_32)
- net A9: now also J8.33 (Pin_33)
- net Clk0: now also J8.37 (Pin_37)
- net Clk2: now also J8.5 (Pin_5)
- net D0: now also U6.22 (D0), J8.9 (Pin_9); no longer U6.15 (D7)
- net D1: now also U6.21 (D1), J8.10 (Pin_10); no longer U6.16 (D6)
- net D2: now also U6.20 (D2), J8.11 (Pin_11); no longer U6.17 (D5)
- net D3: now also U6.19 (D3), J8.12 (Pin_12); no longer U6.18 (D4)
- net D4: now also U6.18 (D4), J8.13 (Pin_13); no longer U6.19 (D3)
- net D5: now also U6.17 (D5), J8.14 (Pin_14); no longer U6.20 (D2)
- net D6: now also U6.16 (D6), J8.15 (Pin_15); no longer U6.21 (D1)
- net D7: now also U6.15 (D7), J8.16 (Pin_16); no longer U6.22 (D0)
- net DISP: now also J8.7 (Pin_7)
- net GND: now also J8.1 (Pin_1), J8.23 (Pin_23)
- net R~{W}: now also J8.6 (Pin_6)
- net ~{PORT}: now also J8.36 (Pin_36)
- net ~{RD}: now also J8.4 (Pin_4)
- net ~{RST}: now also J8.8 (Pin_8)
- net ~{WR}: now also J8.3 (Pin_3)
- new net Q0: J8.17 (Pin_17), J9.1 (Pin_1)
- new net Q1: J8.18 (Pin_18), J9.2 (Pin_2)
- new net Q2: J8.19 (Pin_19), J9.3 (Pin_3)
- new net Q3: J8.20 (Pin_20), J9.4 (Pin_4)
- new net Q4: J8.21 (Pin_21), J9.5 (Pin_5)
- new net Q5: J8.22 (Pin_22), J9.6 (Pin_6)
Other:
- note added: "Mk5"
- moved on the sheet: OSC1
