File: PCB/Mk6/Mk6.kicad_sch (KiCad schematic)
At the start: 2 parts, among them J28 DISPLAY, J5 DISPLAY

Commit message: save point
Parts:
- removed J5: DISPLAY, Connector_PinSocket_2.54mm:PinSocket_1x32_P2.54mm_Vertical, symbol Connector_Generic:Conn_01x32
- J28: value DISPLAY -> EXTENSION
Connections:
- net ~{PORT} renamed ~{IO}

Commit message: save
Parts:
- removed J28: EXTENSION, Connector_PinSocket_2.54mm:PinSocket_1x32_P2.54mm_Vertical, symbol Connector_Generic:Conn_01x32
