File: PCB/Mk6/Mk6.kicad_pcb (KiCad board)
At the start: 2 copper layers, 228.6 x 165.1 mm, 54 parts, among them J10 DISPLAY, J2 Power, J3 Bank, J4 Debug, J5 PortA: 5V PA0 PA1 PA2 PA3 PA4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, J6 PortB: 5V PB0 PB1 PB2 PB3 PB4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, J7 Input Port, J8 Output Port, J9 COM: Gnd,CTS, Vcc, Tx, Rx, DTR, SW2 RESET, U10 R6522, U11 74LS573, U12 74LS574, U2 L7805, U3 DS1813, U4 R65C02, U5 EEPROM, U6 62256, U7 74LS92, U8 GAL20V8B-10, U9 MC68B50, Y2 1.8432 MHz

Commit message: Pre Remap
Parts:
- removed JP1843: 1843, Connector_PinHeader_2.54mm:PinHeader_1x02_P2.54mm_Vertical
- removed JP450: 450, Connector_PinHeader_2.54mm:PinHeader_1x02_P2.54mm_Vertical
- removed JP921: 921, Connector_PinHeader_2.54mm:PinHeader_1x02_P2.54mm_Vertical
- added JP3: 1.8-M-0.9, Connector_PinHeader_2.54mm:PinHeader_1x03_P2.54mm_Vertical, F.Cu at (156.2, 78.7)
- added JP4: 19200 / 9600, Connector_PinHeader_2.54mm:PinHeader_1x03_P2.54mm_Vertical, F.Cu at (185.4, 72.4)
- J4: footprint Connector_PinHeader_2.54mm:PinHeader_1x08_P2.54mm_Vertical -> Connector_PinHeader_2.54mm:PinHeader_1x09_P2.54mm_Vertical
- JP2: value L-ROM-H -> Up-PULL-Down
- moved C7 3.77 mm to (168.9, 78.7)
- moved J4 2.54 mm to (83.8, 139.7)
Connections:
- J4 pad 6: ~{NMI} -> Clk0
- J4 pad 7: /Core/SYNC -> ~{NMI}
- J4 pad 8: +5V -> /Core/SYNC
- U7 pad 8: BaudClk -> Net-(JP4-A)
- U7 pad 9: Net-(JP450-A) -> unconnected-(U7-Q2-Pad9)
Routing:
- net Net-(JP3-B): track 15.9 -> 40.8 mm
- net Net-(JP450-A): track 17.3 -> 0.00 mm
- net Net-(JP4-A): track 0.00 -> 12.3 mm
- net BaudClk: track 58.2 -> 49.8 mm
- net Net-(JP3-A): track 23.9 -> 31.0 mm
- net Clk0: track 129.4 -> 134.6 mm
- net +5V: track 1442.3 -> 1438.5 mm
- net ~{RST}: track 301.3 -> 304.9 mm
- net RDY: track 126.5 -> 129.4 mm
- net Clk2: track 374.5 -> 376.3 mm
- net ~{IRQ}: track 259.6 -> 260.4 mm
- net ~{NMI}: track 239.4 -> 240.2 mm
Other:
- board text added: "4800 / 2400"

Commit message: Added 3-8 IO, extra GAL out, attachment point for !RAM
Parts:
- added J12: ~{RAM} A15, Connector_PinHeader_2.54mm:PinHeader_1x02_P2.54mm_Vertical, F.Cu at (121.9, 76.2)
- added J5: IO:[0,1,2,3,4,5] EXT, Connector_PinSocket_2.54mm:PinSocket_1x07_P2.54mm_Vertical, F.Cu at (160.0, 91.4)
- added U8: 74LS138, Package_DIP:DIP-16_W7.62mm_LongPads, F.Cu at (157.5, 109.2)
- moved J2 14.0 mm to (246.4, 168.9)
- moved C12 10.4 mm to (232.4, 166.4)
- moved JP6 2.54 mm to (250.2, 69.8)
- moved R4 2.54 mm to (242.6, 72.4)
- moved C5 1.27 mm to (168.9, 77.5)
- moved JP3 1.27 mm to (185.4, 71.1)
- renumbered C16 to C10, C12 to C11, C13 to C12, C14 to C13, C2 to C14, C3 to C16, C4 to C2, C5 to C3, C6 to C4, C7 to C5, C8 to C6, C9 to C7, C10 to C8, C11 to C9, J9 to J10, J10 to J11, J5 to J6, J6 to J7, J7 to J8, J8 to J9, JP3 to JP2, JP4 to JP3, JP2 to JP4, JP8 to JP5, JP5 to JP6, JP6 to JP7, JP7 to JP8, U9 to U10, U10 to U11, U11 to U12, U12 to U13, U7 to U4, U4 to U5, U5 to U6, U6 to U7, U8 to U9
Connections:
- RN2 pad 5: DISP -> /Core/EXT
- RN2 pad 6: ~{RD} -> /Core/IO
- RN2 pad 7: ~{WR} -> ~{RD}
- RN2 pad 8: ~{VIA} -> ~{WR}
- RN2 pad 9: ~{COM} -> DISP
- U7 pad 20: A15 -> Net-(J12-A)
- U9 pad 15: ~{COM} -> DISP
- U9 pad 16: ~{VIA} -> ~{WR}
- U9 pad 17: ~{WR} -> ~{RD}
- U9 pad 18: ~{RD} -> /Core/IO
- U9 pad 19: DISP -> /Core/EXT
Routing:
- net ~{IRQ}: track 260.4 -> 333.4 mm
- net GND: track 1256.4 -> 1303.1 mm, vias 20 -> 22
- net A9: track 314.8 -> 357.5 mm, vias 4 -> 6
- net /Core/IO: track 0.00 -> 41.6 mm
- net ~{COM}: track 84.9 -> 46.8 mm
- net /Core/EXT: track 0.00 -> 35.9 mm
- net Net-(J12-A): track 0.00 -> 27.9 mm, vias 0 -> 2
- net BaudClk: track 49.8 -> 76.9 mm
- net A15: track 81.5 -> 55.3 mm, vias 2 -> 0
- net A11: track 346.9 -> 371.7 mm
- net ~{VIA}: track 70.0 -> 49.5 mm
- net A10: track 348.9 -> 366.8 mm
- net +5V: track 1438.5 -> 1451.7 mm, vias 38 -> 40
- net DISP: track 129.1 -> 117.2 mm
- net ~{RD}: track 214.2 -> 203.3 mm
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
Commit message: cleanup
Parts:
- J10: value COM: Gnd,CTS, Vcc, Tx, Rx, DTR -> COM: Gnd, RTS, Vcc, Rx, Tx, DCD-CTS, 5v
- J3: value Bank -> Bank:3..0
- J6: value PortA: 5V PA0 PA1 PA2 PA3 PA4 PA5 PA6 PA7 CA1 CA2 Gnd -> PortA: GND CA2 CA1 PA7 PA6 PA5 PA4 PA3 PA2 PA1 PA0 5v
- J7: value PortB: 5V PB0 PB1 PB2 PB3 PB4 PB5 PB6 PB7 CB1 CB2 Gnd -> PortB: GND CB2 CB1 PB7 PB6 PB5 PB4 PB3 PB2 PB1 PB0 5v
- JP2: value 1.8-M-0.9 -> x1 Osc /2
Routing:
- net ~{ROM}: track 84.7 -> 69.9 mm
- net GND: track 1303.1 -> 1296.0 mm
- net ~{IRQ}: track 333.4 -> 328.5 mm
- net +5V: track 1451.7 -> 1446.9 mm
- net A1: track 325.3 -> 327.8 mm
- net Clk2: track 376.3 -> 378.4 mm
- net R~{W}: track 264.0 -> 266.0 mm
- net DISP: track 117.2 -> 119.0 mm
- net BaudClk: track 76.9 -> 78.7 mm
- net A2: track 323.8 -> 325.6 mm
- net Net-(LCD2-V0): track 59.7 -> 57.9 mm
- net D6: track 381.1 -> 379.6 mm
- net D1: track 338.3 -> 336.8 mm
- net D2: track 332.7 -> 331.2 mm
- net D4: track 377.8 -> 376.3 mm
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