File: PCB/Mk6/power.kicad_sch (KiCad schematic)
At the start: 24 parts, among them J2 Power, SW2 RESET, U2 L7805, U3 DS1813, U7 74LS92, Y2 1.8432 MHz

Commit message: Added 3-8 IO, extra GAL out, attachment point for !RAM
Parts:
- renumbered C16 to C10, C12 to C11, C13 to C12, C14 to C13, C2 to C14, C3 to C16, C4 to C2, C5 to C3, C6 to C4, C7 to C5, C8 to C6, C9 to C7, C10 to C8, C11 to C9, JP3 to JP2, JP4 to JP3, U7 to U4
Changed lines of the file:
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@@
 		(dnp no)
 		(fields_autoplaced yes)
-		(property "Reference" "#PWR04"
+		(property "Reference" "#PWR05"
 			(at 92.71 53.34 0)
 			(effects
@@
 			(project "Mk6"
 				(path "/d41350ce-2040-418d-ae11-f076a5474776/c466e200-7308-4cbf-9cc6-0d7b021a89f4"
-					(reference "#PWR04")
+					(reference "#PWR05")
 					(unit 1)
 				)
@@
 		(on_board yes)
 		(dnp no)
-		(property "Reference" "JP3"
+		(property "Reference" "JP2"
 			(at 152.908 62.484 0)
 			(effects
@@
 			(project "Mk6"
 				(path "/d41350ce-2040-418d-ae11-f076a5474776/c466e200-7308-4cbf-9cc6-0d7b021a89f4"
-					(reference "JP3")
+					(reference "JP2")
 					(unit 1)
 				)
@@
 		(on_board yes)
 		(dnp no)
-		(property "Reference" "C5"
+		(property "Reference" "C3"
 			(at 101.6 34.29 0)
 			(effects
@@
 			(project "Mk6"
 				(path "/d41350ce-2040-418d-ae11-f076a5474776/c466e200-7308-4cbf-9cc6-0d7b021a89f4"
-					(reference "C5")
+					(reference "C3")
 					(unit 1)
 				)
@@
 		(on_board yes)
 		(dnp no)
-		(property "Reference" "C7"
+		(property "Reference" "C5"
 			(at 119.38 34.29 0)
 			(effects
@@
 			(project "Mk6"
 				(path "/d41350ce-2040-418d-ae11-f076a5474776/c466e200-7308-4cbf-9cc6-0d7b021a89f4"
-					(reference "C7")
+					(reference "C5")
 					(unit 1)
 				)
@@
 		(on_board yes)
 		(dnp no)
-		(property "Reference" "C13"
+		(property "Reference" "C12"
 			(at 41.91 37.5538 0)
 			(effects
@@
 			(project "Mk6"
 				(path "/d41350ce-2040-418d-ae11-f076a5474776/c466e200-7308-4cbf-9cc6-0d7b021a89f4"
-					(reference "C13")
+					(reference "C12")
 					(unit 1)
 				)
@@
 		(on_board yes)
 		(dnp no)
-		(property "Reference" "#PWR08"
+		(property "Reference" "#PWR09"
 			(at 81.28 95.25 0)
 			(effects
@@
 			(project "Mk6"
 				(path "/d41350ce-2040-418d-ae11-f076a5474776/c466e200-7308-4cbf-9cc6-0d7b021a89f4"
-					(reference "#PWR08")
+					(reference "#PWR09")
 					(unit 1)
 				)
@@
 		(dnp no)
 		(fields_autoplaced yes)
-		(property "Reference" "#PWR05"
+		(property "Reference" "#PWR04"
 			(at 34.29 53.34 0)
 			(effects
@@
 			(project "Mk6"
 				(path "/d41350ce-2040-418d-ae11-f076a5474776/c466e200-7308-4cbf-9cc6-0d7b021a89f4"
-					(reference "#PWR05")
+					(reference "#PWR04")
 					(unit 1)
 				)
@@
 		(on_board yes)
 		(dnp no)
-		(property "Reference" "C8"
+		(property "Reference" "C6"
 			(at 128.27 34.29 0)
 			(effects
@@
 			(project "Mk6"
 				(path "/d41350ce-2040-418d-ae11-f076a5474776/c466e200-7308-4cbf-9cc6-0d7b021a89f4"
-					(reference "C8")
+					(reference "C6")
 					(unit 1)
 				)
@@
 		(dnp no)
 		(fields_autoplaced yes)
-		(property "Reference" "U7"
+		(property "Reference" "U4"
 			(at 129.1433 64.77 0)
 			(effects
@@
 			(project ""
 				(path "/d41350ce-2040-418d-ae11-f076a5474776/c466e200-7308-4cbf-9cc6-0d7b021a89f4"
-					(reference "U7")
+					(reference "U4")
 					(unit 1)
 				)
@@
 		(on_board yes)
 		(dnp no)
-		(property "Reference" "C6"
+		(property "Reference" "C4"
 			(at 110.49 34.29 0)
 			(effects
@@
 			(project "Mk6"
 				(path "/d41350ce-2040-418d-ae11-f076a5474776/c466e200-7308-4cbf-9cc6-0d7b021a89f4"
-					(reference "C6")
+					(reference "C4")
 					(unit 1)
 				)
@@
 		(on_board yes)
 		(dnp no)
-		(property "Reference" "C9"
+		(property "Reference" "C7"
 			(at 137.16 34.29 0)
 			(effects
@@
 			(project "Mk6"
 				(path "/d41350ce-2040-418d-ae11-f076a5474776/c466e200-7308-4cbf-9cc6-0d7b021a89f4"
-					(reference "C9")
+					(reference "C7")
 					(unit 1)
 				)
@@
 		(on_board yes)
 		(dnp no)
-		(property "Reference" "C16"
+		(property "Reference" "C10"
 			(at 164.338 34.29 0)
 			(effects
@@
 			(project "Mk6"
 				(path "/d41350ce-2040-418d-ae11-f076a5474776/c466e200-7308-4cbf-9cc6-0d7b021a89f4"
-					(reference "C16")
+					(reference "C10")
 					(unit 1)
 				)
@@
 		(on_board yes)
 		(dnp no)
-		(property "Reference" "C4"
+		(property "Reference" "C2"
 			(at 92.71 34.29 0)
 			(effects
@@
 			(project "Mk6"
 				(path "/d41350ce-2040-418d-ae11-f076a5474776/c466e200-7308-4cbf-9cc6-0d7b021a89f4"
-					(reference "C4")
+					(reference "C2")
 					(unit 1)
 				)
@@
 		(on_board yes)
 		(dnp no)
-		(property "Reference" "C10"
+		(property "Reference" "C8"
 			(at 146.05 34.29 0)
 			(effects
@@
 			(project "Mk6"
 				(path "/d41350ce-2040-418d-ae11-f076a5474776/c466e200-7308-4cbf-9cc6-0d7b021a89f4"
-					(reference "C10")
+					(reference "C8")
 					(unit 1)
 				)
@@
 		(on_board yes)
 		(dnp no)
-		(property "Reference" "C3"
+		(property "Reference" "C16"
 			(at 25.4 73.66 0)
 			(effects
@@
 			(project "Mk6"
 				(path "/d41350ce-2040-418d-ae11-f076a5474776/c466e200-7308-4cbf-9cc6-0d7b021a89f4"
-					(reference "C3")
+					(reference "C16")
 					(unit 1)
 				)
@@
 		(on_board yes)
 		(dnp no)
-		(property "Reference" "C14"
+		(property "Reference" "C13"
 			(at 58.928 37.592 0)
 			(effects
@@
 			(project "Mk6"
 				(path "/d41350ce-2040-418d-ae11-f076a5474776/c466e200-7308-4cbf-9cc6-0d7b021a89f4"
-					(reference "C14")
+					(reference "C13")
 					(unit 1)
 				)
@@
 		(on_board yes)
 		(dnp no)
-		(property "Reference" "C2"
+		(property "Reference" "C14"
 			(at 65.024 36.83 0)
 			(effects
@@
 			(project "Mk6"
 				(path "/d41350ce-2040-418d-ae11-f076a5474776/c466e200-7308-4cbf-9cc6-0d7b021a89f4"
-					(reference "C2")
+					(reference "C14")
 					(unit 1)
 				)
@@
 		(on_board yes)
 		(dnp no)
-		(property "Reference" "#PWR09"
+		(property "Reference" "#PWR010"
 			(at 36.83 97.79 0)
 			(effects
@@
 			(project "Mk6"
 				(path "/d41350ce-2040-418d-ae11-f076a5474776/c466e200-7308-4cbf-9cc6-0d7b021a89f4"
-					(reference "#PWR09")
+					(reference "#PWR010")
 					(unit 1)
 				)
@@
 		(on_board yes)
 		(dnp no)
-		(property "Reference" "C12"
+		(property "Reference" "C11"
 			(at 175.26 34.29 0)
 			(effects
@@
 			(project "Mk6"
 				(path "/d41350ce-2040-418d-ae11-f076a5474776/c466e200-7308-4cbf-9cc6-0d7b021a89f4"
-					(reference "C12")
+					(reference "C11")
 					(unit 1)
 				)
@@
 		(on_board yes)
 		(dnp no)
-		(property "Reference" "#PWR07"
+		(property "Reference" "#PWR08"
 			(at 81.28 69.85 0)
 			(effects
@@
 			(project "Mk6"
 				(path "/d41350ce-2040-418d-ae11-f076a5474776/c466e200-7308-4cbf-9cc6-0d7b021a89f4"
-					(reference "#PWR07")
+					(reference "#PWR08")
 					(unit 1)
 				)
@@
 		(on_board yes)
 		(dnp no)
-		(property "Reference" "#PWR019"
+		(property "Reference" "#PWR07"
 			(at 127 68.58 0)
 			(effects
@@
 			(project "Mk6"
 				(path "/d41350ce-2040-418d-ae11-f076a5474776/c466e200-7308-4cbf-9cc6-0d7b021a89f4"
-					(reference "#PWR019")
+					(reference "#PWR07")
 					(unit 1)
 				)
@@
 		(on_board yes)
 		(dnp no)
-		(property "Reference" "JP4"
+		(property "Reference" "JP3"
 			(at 152.908 82.804 0)
 			(effects
@@
 			(project "Mk6"
 				(path "/d41350ce-2040-418d-ae11-f076a5474776/c466e200-7308-4cbf-9cc6-0d7b021a89f4"
-					(reference "JP4")
+					(reference "JP3")
 					(unit 1)
 				)
@@
 		(on_board yes)
 		(dnp no)
-		(property "Reference" "#PWR018"
+		(property "Reference" "#PWR011"
 			(at 127 99.06 0)
 			(effects
@@
 			(project "Mk6"
 				(path "/d41350ce-2040-418d-ae11-f076a5474776/c466e200-7308-4cbf-9cc6-0d7b021a89f4"
-					(reference "#PWR018")
+					(reference "#PWR011")
 					(unit 1)
 				)
@@
 		(on_board yes)
 		(dnp no)
-		(property "Reference" "C11"
+		(property "Reference" "C9"
 			(at 155.448 34.29 0)
 			(effects
@@
 			(project "Mk6"
 				(path "/d41350ce-2040-418d-ae11-f076a5474776/c466e200-7308-4cbf-9cc6-0d7b021a89f4"
-					(reference "C11")
-					(unit 1)
-				)
+					(reference "C9")
+					(unit 1)
+				)

Commit message: cleanup
Parts:
- JP2: value 1.8-M-0.9 -> x1 Osc /2
Changed lines of the file:
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@@
 			)
 		)
-		(property "Value" "1.8-M-0.9"
-			(at 146.304 66.04 0)
+		(property "Value" "x1 Osc /2"
+			(at 157.988 70.612 90)
 			(effects
 				(font
